File: NixieModule_IN-12/Nixie_Module_IN-12.kicad_pcb (KiCad board)
At the start: 2 copper layers, 20 x 40 mm, 43 parts, among them J1 CONN_01X07, J3 CONN_01X02, J4 CONN_01X02, Q1 Q_NPN_BEC, Q10 Q_NPN_BEC, Q11 Q_NPN_BEC, Q2 Q_NPN_BEC, Q3 Q_NPN_BEC, Q4 Q_NPN_BEC, Q5 Q_NPN_BEC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

Commit message: Update documentation
Parts:
- removed LED1: VAL**, WS2812b:WS2812B
- added U1: SK6812mini, FidgetSpinner:SK6812MINI, F.Cu at (79.2, 91.9)
- R1: value 15k -> R
- R14, R15, R16, R17, R18, R19, R2: value 10k -> R
Routing:
- net +5V: track 49.0 -> 51.3 mm, vias 4 -> 3
- net GND: vias 30 -> 31
