File: NixieModule_IN-14/Nixie_Module_IN-14.sch (KiCad schematic (older format))
At the start: 41 parts, among them J3 CONN_01X02, Q1 Q_NPN_BEC, Q10 Q_NPN_BEC, Q2 Q_NPN_BEC, Q3 Q_NPN_BEC, Q4 Q_NPN_BEC, Q5 Q_NPN_BEC, Q6 Q_NPN_BEC, Q7 Q_NPN_BEC, Q8 Q_NPN_BEC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

Commit message: Update documentation
Parts:
- C1, C2: symbol device:C -> Device:C
- C3: value 47u -> 4.7u; symbol device:C -> Device:C
- Q1, Q10, Q2, Q3, Q4, Q5, Q6, Q7, Q8, Q9: symbol device:Q_NPN_BEC -> Device:Q_NPN_BEC
- R1: value 15k -> 47k; symbol device:R -> Device:R
- R10, R11, R12, R14, R15, R16, R17, R18, R19, R2, R3, R4, R5, R6, R7, R8, R9: symbol device:R -> Device:R
Changed lines of the file:
@@
 $EndDescr
 $Comp
-L device:R R1
+L Device:R R1
 U 1 1 5B6A64B0
 P 2550 1650
 F 0 "R1" V 2630 1650 50  0000 C CNN
-F 1 "15k" V 2550 1650 50  0000 C CNN
+F 1 "47k" V 2550 1650 50  0000 C CNN
 F 2 "R_SMD:R_0603" V 2480 1650 50  0001 C CNN
 F 3 "" H 2550 1650 50  0001 C CNN
@@
 I2C_SDA
 $Comp
-L device:C C1
+L Device:C C1
 U 1 1 5B6B5DDE
 P 1900 5750
@@
 $EndComp
 $Comp
-L device:C C2
+L Device:C C2
 U 1 1 5B6B6351
 P 2150 5750
@@
 ADDR_3
 $Comp
-L device:Q_NPN_BEC Q1
+L Device:Q_NPN_BEC Q1
 U 1 1 5B7F7F44
 P 4900 1700
@@
 $EndComp
 $Comp
-L device:Q_NPN_BEC Q3
+L Device:Q_NPN_BEC Q3
 U 1 1 5B7F8009
 P 6000 1700
@@
 $EndComp
 $Comp
-L device:Q_NPN_BEC Q5
+L Device:Q_NPN_BEC Q5
 U 1 1 5B7F8093
 P 7200 1700
@@
 $EndComp
 $Comp
-L device:Q_NPN_BEC Q7
+L Device:Q_NPN_BEC Q7
 U 1 1 5B7F810D
 P 8700 1700
@@
 $EndComp
 $Comp
-L device:Q_NPN_BEC Q9
+L Device:Q_NPN_BEC Q9
 U 1 1 5B7F817C
 P 10200 1700
@@
 $EndComp
 $Comp
-L device:Q_NPN_BEC Q2
+L Device:Q_NPN_BEC Q2
 U 1 1 5B7F82DA
 P 5650 3500
@@
 $EndComp
 $Comp
-L device:Q_NPN_BEC Q4
+L Device:Q_NPN_BEC Q4
 U 1 1 5B7F8359
 P 6900 3500
@@
 $EndComp
 $Comp
-L device:Q_NPN_BEC Q6
+L Device:Q_NPN_BEC Q6
 U 1 1 5B7F83D9
 P 8050 3500
@@
 $EndComp
 $Comp
-L device:Q_NPN_BEC Q8
+L Device:Q_NPN_BEC Q8
 U 1 1 5B7F8458
 P 9350 3500
@@
 $EndComp
 $Comp
-L device:Q_NPN_BEC Q10
+L Device:Q_NPN_BEC Q10
 U 1 1 5B7F84E2
 P 10550 3500
@@
 $EndComp
 $Comp
-L device:R R3
+L Device:R R3
 U 1 1 5B7FACAB
 P 4550 1700
@@
 $EndComp
 $Comp
-L device:R R5
+L Device:R R5
 U 1 1 5B7FB4A4
 P 5650 1700
@@
 $EndComp
 $Comp
-L device:R R7
+L Device:R R7
 U 1 1 5B7FB9AA
 P 6850 1700
@@
 $EndComp
 $Comp
-L device:R R9
+L Device:R R9
 U 1 1 5B7FBC40
 P 8350 1700
@@
 $EndComp
 $Comp
-L device:R R11
+L Device:R R11
 U 1 1 5B7FBEBB
 P 9850 1700
@@
 $EndComp
 $Comp
-L device:R R4
+L Device:R R4
 U 1 1 5B7FC473
 P 5300 3500
@@
 $EndComp
 $Comp
-L device:R R6
+L Device:R R6
 U 1 1 5B7FC50B
 P 6550 3500
@@
 $EndComp
 $Comp
-L device:R R8
+L Device:R R8
 U 1 1 5B7FC94D
 P 7700 3500
@@
 $EndComp
 $Comp
-L device:R R10
+L Device:R R10
 U 1 1 5B7FCB6D
 P 9000 3500
@@
 $EndComp
 $Comp
-L device:R R12
+L Device:R R12
 U 1 1 5B7FCC87
 P 10200 3500
@@
 ADDR_0
 $Comp
-L device:R R14
+L Device:R R14
 U 1 1 5B8C85A7
 P 6550 5250
@@
 \nPC9685 Address Config Hadware Strap\nALL CALL ADDR: 0xE0\nSOFTWARE RESET ADDR: 0x06
 $Comp
-L device:R R15
+L Device:R R15
 U 1 1 5B8EB4E0
 P 6550 5450
@@
 $EndComp
 $Comp
-L device:R R16
+L Device:R R16
 U 1 1 5B8EB538
 P 6550 5650
@@
 $EndComp
 $Comp
-L device:R R17
+L Device:R R17
 U 1 1 5B8EB592
 P 6550 5850
@@
 	3300 5700 3300 5750
 $Comp
-L device:R R2
+L Device:R R2
 U 1 1 5B916675
 P 3300 5900
@@
 	1400 3900 1400 3800
 $Comp
-L device:C C3
+L Device:C C3
 U 1 1 5B9866E4
 P 1000 4050
 F 0 "C3" H 1025 4150 50  0000 L CNN
-F 1 "47u" H 1025 3950 50  0000 L CNN
+F 1 "4.7u" H 1025 3950 50  0000 L CNN
 F 2 "C_SMD:C_0603" H 1038 3900 50  0001 C CNN
 F 3 "" H 1000 4050 50  0001 C CNN
@@
 	5050 6400 5250 6400
 $Comp
-L device:R R18
+L Device:R R18
 U 1 1 5BA01E66
 P 8750 5200
@@
 $EndComp
 $Comp
-L device:R R19
+L Device:R R19
 U 1 1 5BA0204E
 P 8900 5200

Commit message: Document update
Parts:
- gave numbers to parts that had none: 3
Changed lines of the file:
@@
 EESchema Schematic File Version 4
 LIBS:Nixie_Module_IN-14-cache
-EELAYER 26 0
+EELAYER 29 0
 EELAYER END
 $Descr A4 11693 8268
@@
 $EndComp
 $Comp
-L NixieModule:SK6812mini U?
+L NixieModule:SK6812mini U1
 U 1 1 5C571FF8
 P 2050 3750
-F 0 "U?" H 2050 3847 60  0000 C CNN
+F 0 "U1" H 2050 3847 60  0000 C CNN
 F 1 "SK6812mini" H 2050 3741 60  0000 C CNN
 F 2 "" H 2050 3750 60  0000 C CNN
@@
 $EndComp
 $Comp
-L conn:Conn_01x07_Female J?
+L conn:Conn_01x07_Female J1
 U 1 1 5C5723A7
 P 9600 5650
-F 0 "J?" H 9627 5676 50  0000 L CNN
+F 0 "J1" H 9627 5676 50  0000 L CNN
 F 1 "Conn_01x07_Female" H 9627 5585 50  0000 L CNN
 F 2 "" H 9600 5650 50  0001 C CNN
@@
 $EndComp
 $Comp
-L conn:Conn_01x02_Female J?
+L conn:Conn_01x02_Female J2
 U 1 1 5C5726E4
 P 10650 5800
-F 0 "J?" H 10677 5776 50  0000 L CNN
+F 0 "J2" H 10677 5776 50  0000 L CNN
 F 1 "Conn_01x02_Female" H 10677 5685 50  0000 L CNN
 F 2 "" H 10650 5800 50  0001 C CNN
